Commit message: Updating Robot URDF features...

File: urdf/my_robot.urdf (robot description, URDF)
Before this commit: robot my_robot, 3 links, 2 joints
Links:
- removed link second_link
- removed link third_link
- added link base_footprint_link
- added link caster_wheel_link; visual sphere radius=0.05
- added link left_wheel_link; visual cylinder length=0.05 radius=0.1
- added link right_wheel_link; visual cylinder length=0.05 radius=0.1
Joints:
- removed joint base_second_joint
- removed joint second_third_joint
- added joint base_caster_wheel_joint: type fixed, parent base_link, child caster_wheel_link, origin xyz=0.2 0 -0.05 rpy=0 0 0
- added joint base_joint: type fixed, parent base_footprint_link, child base_link, origin xyz=0 0 0.1 rpy=0 0 0
- added joint base_left_wheel_joint: type continuous, parent base_link, child left_wheel_link, origin xyz=-0.15 0.225 0 rpy=0 0 0, axis 0 1 0
- added joint base_rigth_wheel_joint: type continuous, parent base_link, child right_wheel_link, origin xyz=-0.15 -0.225 0 rpy=0 0 0, axis 0 1 0
